Commit message: Kamera yeri güncellendi

File: src/sadit_description/urdf/d435_camera2.xacro (robot description, xacro)
@@ -151,6 +151,6 @@
           <camera_name>${name}_depth</camera_name>
           <frame_name>${name}_depth_optical_frame</frame_name>
-          <image_topic_name>sadit/camera/depth/image_raw</image_topic_name>
-          <camera_info_topic_name>sadit/camera/depth/camera_info</camera_info_topic_name>
+          <image_topic_name>sadit/camera2/depth/image_raw</image_topic_name>
+          <camera_info_topic_name>sadit/camera2/depth/camera_info</camera_info_topic_name>
         </plugin>
       </sensor>
@@ -180,7 +180,7 @@
           <camera_name>${name}_points</camera_name>
           <frame_name>${name}_depth_optical_frame</frame_name>
-          <point_cloud_topic_name>sadit/camera/depth/color/points</point_cloud_topic_name>
-          <image_topic_name>sadit/camera/depth/image_rect_raw</image_topic_name>
-          <camera_info_topic_name>sadit/camera/depth/camera_info</camera_info_topic_name>
+          <point_cloud_topic_name>sadit/camera2/depth/color/points</point_cloud_topic_name>
+          <image_topic_name>sadit/camera2/depth/image_rect_raw</image_topic_name>
+          <camera_info_topic_name>sadit/camera2/depth/camera_info</camera_info_topic_name>
           <point_cloud_cutoff>0.1</point_cloud_cutoff>
           <point_cloud_cutoff_max>10.0</point_cloud_cutoff_max>

File: src/sadit_description/urdf/sadit.xacro (robot description, xacro)
@@ -35,5 +35,5 @@
 <xacro:d435_gazebo_plugins name="camera"/>
 <!-- Kamera (D435) -->
-<xacro:realsense_d435_2 parent="base_link" name="camera2" xyz="-0.8 0.15 0.25" rpy="0 0.416666667 3.14159"/>
+<xacro:realsense_d435_2 parent="camera2_mount_link" name="camera2" xyz="0 0 0" rpy="0 0 0"/>
 <xacro:d435_gazebo_plugins_2 name="camera2"/>
 <!-- IMU Sensor -->
@@ -119,4 +119,5 @@
   </collision>
 </link>
+<link name="camera2_mount_link"/>
 <joint name="sol_on" type="continuous">
   <origin xyz="0.0825 0.073 -0.048" rpy="0 0 0"/>
@@ -143,3 +144,8 @@
   <axis xyz="0.0 -1.0 0.0"/>
 </joint>
+<joint name="camera2_mount_joint" type="fixed">
+  <parent link="base_link"/>
+  <child link="camera2_mount_link"/>
+  <origin xyz="-0.02 0.25 0.1" rpy="0 0 3.14159"/>
+</joint>
 </robot>
